Commit message: Update stella.urdf

File: stella_description/urdf/stella.urdf (robot description, URDF)
Before this commit: robot stella, 4 links, 3 joints
Links:
- link base_link: mass 7.18 -> 1.47; geometry collision box size=0.17 0.207 0.164; visual mesh filename=package://stella_description/meshes/bases/STELLA-N1.stl scale=0.001 0.001 0.001
Joints:
- joint imu_joint: origin xyz=0.0 0.0 0.071 rpy=0.0 0.0 0.0 -> xyz=-0.06 0.0 0.063 rpy=0.0 0.0 0.0
- joint scan_joint: origin xyz=0.145 0.0 0.229 rpy=0.0 0.0 0.0 -> xyz=0.06 0.0 0.14 rpy=0.0 0.0 0.0

Commit message: Update stella.urdf

File: stella_description/urdf/stella.urdf (robot description, URDF)
Before this commit: robot stella, 4 links, 3 joints
Links:
- link base_link: geometry collision box size=0.17 0.207 0.164; visual mesh filename=package://stella_description/meshes/bases/STELLA-N2.stl scale=0.001 0.001 0.001
